Commit message: add mrobot

File: urdf/accessory/imu.xacro (robot description, xacro)
@@ -3,4 +3,9 @@
     <xacro:macro name="imu" params="ns">
         <link name="$(arg ns)/imu_link">
+            <inertial>
+                <mass value="1e-5" />
+                <origin xyz="0 0 0" rpy="0 0 0" />
+                <inertia ixx="1e-6" ixy="0" ixz="0" iyy="1e-6" iyz="0" izz="1e-6" />
+            </inertial>
             <visual>
                 <origin xyz="0 0 0" rpy="0 0 0" />
@@ -9,9 +14,4 @@
                 </geometry>
             </visual>
-            <inertial>
-                <mass value="1e-5" />
-                <origin xyz="0 0 0" rpy="0 0 0" />
-                <inertia ixx="1e-6" ixy="0" ixz="0" iyy="1e-6" iyz="0" izz="1e-6" />
-            </inertial>
         </link>
         <gazebo reference="$(arg ns)/imu_link">

File: urdf/accessory/rplidar.xacro (robot description, xacro)
@@ -6,7 +6,5 @@
                 <mass value="0.1" />
                 <origin xyz="0 0 0" />
-                <inertia ixx="0.01" ixy="0.0" ixz="0.0"
-                         iyy="0.01" iyz="0.0"
-                         izz="0.01" />
+                <inertia ixx="0.01" ixy="0.0" ixz="0.0" iyy="0.01" iyz="0.0" izz="0.01" />
             </inertial>
             <visual>
@@ -15,12 +13,5 @@
                     <cylinder length="0.05" radius="0.02"/>
                 </geometry>
-                <material name="gray"/>
             </visual>
-            <collision>
-                <origin xyz="0 0 0" rpy="0 0 0" />
-                <geometry>
-                    <cylinder length="0.05" radius="0.02"/>
-                </geometry>
-            </collision>
         </link>
         <gazebo reference="$(arg ns)/rplidar_link">
@@ -53,5 +44,5 @@
                 </ray>
                 <plugin name="gazebo_rplidar" filename="libgazebo_ros_laser.so">
-                    <topicName>$(arg ns)/scan</topicName>
+                    <topicName>scan</topicName>
                     <frameName>$(arg ns)/rplidar_link</frameName>
                 </plugin>

File: urdf/accessory/usb_camera.xacro (robot description, xacro)
@@ -1,6 +1,6 @@
 <?xml version="1.0" encoding="utf-8"?>
 <robot xmlns:xacro="http://www.ros.org/wiki/xacro">
-    <xacro:macro name="usb_camera" params="prefix:=camera">
-        <link name="${prefix}_link">
+    <xacro:macro name="usb_camera" params="ns">
+        <link name="$(arg ns)/camera_link">
             <visual>
                 <origin xyz="0 0 0" rpy="0 0 0" />
@@ -15,8 +15,8 @@
             </inertial>
         </link>
-        <gazebo reference="${prefix}_link">
+        <gazebo reference="$(arg ns)/camera_link">
             <material>Gazebo/Black</material>
         </gazebo>
-        <gazebo reference="camera_link">
+        <gazebo reference="$(arg ns)/camera_link">
             <sensor type="camera" name="camera_node">
                 <update_rate>30.0</update_rate>
@@ -24,16 +24,16 @@
                     <horizontal_fov>1.3962634</horizontal_fov>
                     <image>
-                        <width>800</width>
-                        <height>600</height>
-                        <format>R8G8B8</format>
+                    <width>800</width>
+                    <height>600</height>
+                    <format>R8G8B8</format>
                     </image>
                     <clip>
-                        <near>0.02</near>
-                        <far>300</far>
+                    <near>0.02</near>
+                    <far>300</far>
                     </clip>
                     <noise>
-                        <type>gaussian</type>
-                        <mean>0.0</mean>
-                        <stddev>0.007</stddev>
+                    <type>gaussian</type>
+                    <mean>0.0</mean>
+                    <stddev>0.007</stddev>
                     </noise>
                 </camera>
@@ -44,5 +44,5 @@
                     <cameraInfoTopicName>camera_info</cameraInfoTopicName>
                     <cameraName>camera</cameraName>
-                    <frameName>camera_link</frameName>
+                    <frameName>camera_frame</frameName>
                     <hackBaseline>0.07</hackBaseline>
                     <distortionK1>0.0</distortionK1>

File: urdf/leo_rover/main.xacro (robot description, xacro)
@@ -1,11 +1,11 @@
 <?xml version="1.0" encoding="utf-8"?>
-<robot xmlns:xacro="http://www.ros.org/wiki/xacro"
-       name="leo_rover">
+<robot xmlns:xacro="http://www.ros.org/wiki/xacro" name="leo_rover">
   <xacro:arg name="tf_odom_enabled" default="true" />
   <xacro:arg name="ns" default="" />
   <!-- include -->
   <xacro:include filename="$(find ros_my_robot_gazebo)/urdf/leo_rover/wheel.xacro" />
-  <xacro:include filename="$(find ros_my_robot_gazebo)/urdf/leo_rover/imu.xacro" />
-  <xacro:include filename="$(find ros_my_robot_gazebo)/urdf/leo_rover/rplidar.xacro" />
+  <xacro:include filename="$(find ros_my_robot_gazebo)/urdf/accessory/imu.xacro" />
+  <xacro:include filename="$(find ros_my_robot_gazebo)/urdf/accessory/rplidar.xacro" />
+  <xacro:include filename="$(find ros_my_robot_gazebo)/urdf/accessory/usb_camera.xacro" />
   <!-- global vars -->
   <xacro:property name="M_PI" value="3.1415926535897931" />
@@ -28,8 +28,4 @@
   </gazebo>
   <!-- wheel -->
-  <xacro:wheel ns="(arg ns)" name="FL" model="left" mu1="5.0" mu2="2.0" />
-  <xacro:wheel ns="(arg ns)" name="FR" model="right" mu1="5.0" mu2="2.0" />
-  <xacro:wheel ns="(arg ns)" name="RL" model="left" mu1="0.0" mu2="0.0" />
-  <xacro:wheel ns="(arg ns)" name="RR" model="right" mu1="0.0" mu2="0.0" />
   <joint name="$(arg ns)/wheel_FL_joint" type="continuous">
     <origin xyz="0.1472 0.1114 -0.1353" rpy="0 0 ${pi}"/>
@@ -38,4 +34,5 @@
     <axis xyz="0 -1 0"/>
   </joint>
+  <xacro:wheel ns="(arg ns)" name="FL" model="left" mu1="5.0" mu2="2.0" />
   <joint name="$(arg ns)/wheel_FR_joint" type="continuous">
     <origin xyz="0.1472 -0.1114 -0.1353" rpy="0 0 0"/>
@@ -44,4 +41,5 @@
     <axis xyz="0 1 0"/>
   </joint>
+  <xacro:wheel ns="(arg ns)" name="FR" model="right" mu1="5.0" mu2="2.0" />
   <joint name="$(arg ns)/wheel_RL_joint" type="continuous">
     <origin xyz="-0.1419 0.1114 -0.1353" rpy="0 0 ${pi}"/>
@@ -50,4 +48,5 @@
     <axis xyz="0 -1 0"/>
   </joint>
+  <xacro:wheel ns="(arg ns)" name="RL" model="left" mu1="0.0" mu2="0.0" />
   <joint name="$(arg ns)/wheel_RR_joint" type="continuous">
     <origin xyz="-0.1419 -0.1114 -0.1353" rpy="0 0 0"/>
@@ -56,11 +55,12 @@
     <axis xyz="0 1 0"/>
   </joint>
-  <!-- camera -->
-  <link name="$(arg ns)/camera_frame"/>
+  <xacro:wheel ns="(arg ns)" name="RR" model="right" mu1="0.0" mu2="0.0" />
+  <!-- usb_camera -->
   <joint name="$(arg ns)/camera_joint" type="fixed">
     <origin xyz="0.0971 0 -0.0427" rpy="0 0 0"/>
     <parent link="$(arg ns)/base_link"/>
-    <child link="$(arg ns)/camera_frame"/>
+    <child link="$(arg ns)/camera_link"/>
   </joint>
+  <xacro:usb_camera ns="$(arg ns)" />
   <!-- rplidar -->
   <joint name="$(arg ns)/rplidar_joint" type="fixed">
@@ -77,40 +77,11 @@
   </joint>
   <xacro:imu ns="$(arg ns)" />
-  <!-- camera -->
-  <gazebo reference="camera_frame">
-    <sensor type="camera" name="camera_node">
-      <update_rate>30.0</update_rate>
-      <camera name="head">
-        <horizontal_fov>1.3962634</horizontal_fov>
-        <image>
-          <width>800</width>
-          <height>600</height>
-          <format>R8G8B8</format>
-        </image>
-        <clip>
-          <near>0.02</near>
-          <far>300</far>
-        </clip>
-        <noise>
-          <type>gaussian</type>
-          <mean>0.0</mean>
-          <stddev>0.007</stddev>
-        </noise>
-      </camera>
-      <plugin name="gazebo_camera" filename="libgazebo_ros_camera.so">
-        <alwaysOn>true</alwaysOn>
-        <updateRate>0.0</updateRate>
-        <imageTopicName>image_raw</imageTopicName>
-        <cameraInfoTopicName>camera_info</cameraInfoTopicName>
-        <cameraName>camera</cameraName>
-        <frameName>camera_frame</frameName>
-        <hackBaseline>0.07</hackBaseline>
-        <distortionK1>0.0</distortionK1>
-        <distortionK2>0.0</distortionK2>
-        <distortionK3>0.0</distortionK3>
-        <distortionT1>0.0</distortionT1>
-        <distortionT2>0.0</distortionT2>
-      </plugin>
-    </sensor>
+  <!-- joint state -->
+  <gazebo>
+    <plugin name="gazebo_ros_control" filename="libgazebo_ros_control.so">
+      <robotNamespace>$(arg ns)</robotNamespace>
+      <robotSimType>gazebo_ros_control/DefaultRobotHWSim</robotSimType>
+      <legacyModeNS>true</legacyModeNS>
+    </plugin>
   </gazebo>
   <!-- skid steering drive -->
@@ -123,6 +94,4 @@
       <leftRearJoint>$(arg ns)/wheel_RL_joint</leftRearJoint>
       <rightRearJoint>$(arg ns)/wheel_RR_joint</rightRearJoint>
-      <wheelSeparation>0.32</wheelSeparation>
-      <wheelDiameter>0.13</wheelDiameter>
       <robotBaseFrame>$(arg ns)/base_link</robotBaseFrame>
       <odometryFrame>$(arg ns)/odom</odometryFrame>
@@ -132,4 +101,6 @@
       <broadcastTF>$(arg tf_odom_enabled)</broadcastTF>
       <torque>30</torque>
+      <wheelSeparation>0.32</wheelSeparation>
+      <wheelDiameter>0.13</wheelDiameter>
       <covariance_x>0.001</covariance_x>
       <covariance_y>0.001</covariance_y>

File: urdf/mrobot/caster.xacro (robot description, xacro)
@@ -2,7 +2,12 @@
 <robot xmlns:xacro="http://www.ros.org/wiki/xacro">
     <!-- Macro for caster joint -->
-    <xacro:macro name="caster" params="fb translateX parent">
+    <xacro:macro name="caster" params="fb translateX parent ns">
         <!-- fb: front, back -->
-        <link name="${fb}_caster_link">
+        <joint name="base_to_${fb}_caster_joint" type="fixed">
+            <origin xyz="${translateX*caster_joint_origin_x} 0 ${-caster_radius}" rpy="0 0 0"/>
+            <parent link="${parent}"/>
+            <child link="$(arg ns)/${fb}_caster_link"/>
+        </joint>
+        <link name="$(arg ns)/${fb}_caster_link">
             <visual>
                 <origin xyz="0 0 0 " rpy="0 0 0" />
@@ -23,9 +28,4 @@
             <material>Gazebo/Gray</material>
         </gazebo>
-        <joint name="base_to_${fb}_caster_joint" type="fixed">
-            <parent link="${parent}"/>
-            <child link="${fb}_caster_link"/>
-            <origin xyz="${translateX*caster_joint_origin_x} 0 ${-caster_radius}" rpy="0 0 0"/>
-        </joint>
     </xacro:macro>
 </robot>

File: urdf/mrobot/plate.xacro (robot description, xacro)
@@ -2,6 +2,11 @@
 <robot xmlns:xacro="http://www.ros.org/wiki/xacro">
     <!-- Macro for plate joint -->
-    <xacro:macro name="plate" params="num parent">
-        <link name="plate_${num}_link">
+    <xacro:macro name="plate" params="num parent ns">
+        <joint name="$(arg ns)/plate_${num}_joint" type="fixed">
+            <origin xyz="0 0 ${plate_height}" rpy="0 0 0" />
+            <parent link="${parent}"/>
+            <child link="$(arg ns)/plate_${num}_link" />
+        </joint>
+        <link name="$(arg ns)/plate_${num}_link">
             <xacro:cylinder_inertial_matrix  m="${plate_mass}" r="${base_link_radius}" h="${base_link_length}" />
             <visual>
@@ -19,12 +24,7 @@
             </collision>
         </link>
-        <gazebo reference="plate_${num}_link">
+        <gazebo reference="$(arg ns)/plate_${num}_link">
             <material>Gazebo/Blue</material>
         </gazebo>
-        <joint name="plate_${num}_joint" type="fixed">
-            <origin xyz="0 0 ${plate_height}" rpy="0 0 0" />
-            <parent link="${parent}"/>
-            <child link="plate_${num}_link" />
-        </joint>
     </xacro:macro>
 </robot>

File: urdf/mrobot/wheel.xacro (robot description, xacro)
@@ -2,7 +2,13 @@
 <robot xmlns:xacro="http://www.ros.org/wiki/xacro">
     <!-- Macro for wheel joint -->
-    <xacro:macro name="wheel" params="lr translateY parent">
+    <xacro:macro name="wheel" params="lr translateY parent ns">
         <!-- lr: left, right -->
-        <link name="wheel_${lr}_link">
+        <joint name="$(arg ns)/wheel_${lr}_joint" type="continuous">
+            <parent link="${parent}"/>
+            <child link="$(arg ns)/wheel_${lr}_link"/>
+            <origin xyz="${motor_x} ${translateY * base_link_radius} 0" rpy="0 0 0" />
+            <axis xyz="0 1 0" rpy="0 0 0" />
+        </joint>
+        <link name="$(arg ns)/wheel_${lr}_link">
             <visual>
                 <origin xyz="0 0 0" rpy="${M_PI/2} 0  0 " />
@@ -20,5 +26,5 @@
             <xacro:cylinder_inertial_matrix  m="${wheel_mass}" r="${wheel_radius}" h="${wheel_height}" />
         </link>
-        <gazebo reference="wheel_${lr}_link">
+        <gazebo reference="$(arg ns)/wheel_${lr}_link">
             <material>Gazebo/Black</material>
             <mu1>5.0</mu1>
@@ -30,10 +36,4 @@
             <fdir1>0 0 0</fdir1>
         </gazebo>
-        <joint name="wheel_${lr}_joint" type="continuous">
-            <parent link="${parent}"/>
-            <child link="wheel_${lr}_link"/>
-            <origin xyz="${motor_x} ${translateY * base_link_radius} 0" rpy="0 0 0" />
-            <axis xyz="0 1 0" rpy="0 0 0" />
-        </joint>
     </xacro:macro>
 </robot>
